File: HW/ESP-01_Prog_SMD/ESP-01.sch (KiCad schematic (older format))
At the start: 5 parts, among them P3 PROG, U1 ESP-01

Commit message: Modify ESP-32 Breakout
Parts:
- P3: symbol CONN_01X06 -> ESP-01-rescue:CONN_01X06
- R1, R2, R3: symbol R_Small -> Device:R_Small
- U1: symbol ESP-01 -> ESP-01-rescue:ESP-01
Changed lines of the file:
@@
-EESchema Schematic File Version 2
-LIBS:power
-LIBS:device
-LIBS:transistors
-LIBS:conn
-LIBS:linear
-LIBS:regul
-LIBS:74xx
-LIBS:cmos4000
-LIBS:adc-dac
-LIBS:memory
-LIBS:xilinx
-LIBS:microcontrollers
-LIBS:dsp
-LIBS:microchip
-LIBS:analog_switches
-LIBS:motorola
-LIBS:texas
-LIBS:intel
-LIBS:audio
-LIBS:interface
-LIBS:digital-audio
-LIBS:philips
-LIBS:display
-LIBS:cypress
-LIBS:siliconi
-LIBS:opto
-LIBS:atmel
-LIBS:contrib
-LIBS:valves
-LIBS:modlib
+EESchema Schematic File Version 4
 LIBS:ESP-01-cache
-EELAYER 25 0
+EELAYER 26 0
 EELAYER END
 $Descr A4 11693 8268
@@
 $EndDescr
 $Comp
-L CONN_01X06 P3
+L ESP-01-rescue:CONN_01X06 P3
 U 1 1 56FE78B6
 P 5750 3950
@@
 $EndComp
 $Comp
-L ESP-01 U1
+L ESP-01-rescue:ESP-01 U1
 U 1 1 56FE7971
 P 5800 2750
@@
 $EndComp
 $Comp
-L R_Small R1
+L Device:R_Small R1
 U 1 1 56FE79C6
 P 5000 2300
@@
 	6600 2800 6300 2800
 Wire Wire Line
-	6600 2150 6600 3300
+	6600 2150 6600 2800
 Wire Wire Line
 	5150 2400 5150 2700
@@
 	5150 2700 5300 2700
 Wire Wire Line
-	5000 2400 5000 3300
+	5000 2400 5000 2800
 Wire Wire Line
 	5000 2800 5300 2800
@@
 Connection ~ 6600 2800
 $Comp
-L GND #PWR01
+L power:GND #PWR01
 U 1 1 56FECE70
 P 6450 3050
@@
 	6450 2600 6450 3050
 $Comp
-L +3.3V #PWR02
+L power:+3.3V #PWR02
 U 1 1 56FECEC8
 P 6600 1900
@@
 $EndComp
 $Comp
-L +3.3V #PWR03
+L power:+3.3V #PWR03
 U 1 1 56FECEF4
 P 5000 2100
@@
 	6600 1950 6600 1900
 $Comp
-L +3.3V #PWR04
+L power:+3.3V #PWR04
 U 1 1 56FED1A9
 P 4850 2750
@@
 	4850 2900 4850 2750
 $Comp
-L GND #PWR05
+L power:GND #PWR05
 U 1 1 56FED283
 P 6200 3900
@@
 	5500 3150 5500 3750
 $Comp
-L R_Small R2
+L Device:R_Small R2
 U 1 1 56FED431
 P 5150 2300
@@
 $EndComp
 $Comp
-L R_Small R3
+L Device:R_Small R3
 U 1 1 56FED53D
 P 6600 2050
@@
 	5700 3300 5700 3750
 $Comp
-L +3.3V #PWR06
+L power:+3.3V #PWR06
 U 1 1 57FB0688
 P 5900 3650
@@
 Wire Wire Line
 	5900 3650 5900 3750
+Wire Wire Line
+	5000 2800 5000 3300
+Wire Wire Line
+	6600 2800 6600 3300
 $EndSCHEMATC
