File: HW/ESP-WROOM-32_Breakout/ESP-WROOM-32_Breakout.sch (KiCad schematic (older format))
At the start: 10 parts, among them P1 CONN_01X06, P2 CONN_01X18, P3 CONN_01X18, U1 ESP32-WROOM

Commit message: Modify ESP-32 Breakout
Connections:
- net GND: now also P1.1 (P1); no longer P1.6 (P6)
- net RXD: now also P1.5 (P5); no longer P1.2 (P2)
- net TXD: now also P1.6 (P6); no longer P1.1 (P1)
- net VCC: now also P1.2 (P2); no longer P1.5 (P5)
- net ~FLASH: now also P1.3 (P3); no longer P1.4 (P4)
- net ~RST: now also P1.4 (P4); no longer P1.3 (P3)
Changed lines of the file:
@@
 F 3 "" H 1700 3150 50  0000 C CNN
 	1    1700 3150
-	-1   0    0    -1
+	-1   0    0    1
 $EndComp
 $Comp
